File: app/services/layout_service/data/temp/project/Project.kicad_pcb (KiCad board)
At the start: 2 copper layers, 40 x 40 mm, 58 parts

Commit message: 流程适配-开始考虑焊盘和旋转
Parts:
- removed IC**: SOT95P285X113-3N, SOT95P285X113-3N
- removed REF** (x4): C_0603_1608Metric, C_0603_1608Metric
- removed REF**: 8L_USON_2X3_ISI, 8L_USON_2X3_ISI
- removed REF** (x2): YAG_CC0603_YAG, YAG_CC0603_YAG
- removed REF** (x2): CAP_0402_SAM, CAP_0402_SAM
- removed REF**: BMX160_BOS, BMX160_BOS
- removed REF**: SOT23-3_LTF, SOT23-3_LTF
- removed REF** (x7): R_0402_1005Metric, R_0402_1005Metric
- removed REF** (x5): C_0402_1005Metric, C_0402_1005Metric
- removed REF**: MC3635_MEM, MC3635_MEM
- removed REF**: SOT25_DIO, SOT25_DIO
- removed REF**: SOD-123_ONS, SOD-123_ONS
- removed REF**: CUI_PJ-044A, CUI_PJ-044A
- removed REF**: SDO_CFP5_SOD128_NEX, SDO_CFP5_SOD128_NEX
- removed REF**: CAP_CL10A105KB8NNN_SAM, CAP_CL10A105KB8NNN_SAM
- removed REF**: SOT-23_DIO, SOT-23_DIO
- removed REF**: SOT-323_DIO, SOT-323_DIO
- removed REF**: R_0603_1608Metric, R_0603_1608Metric
- removed REF**: SOT-23_MC_MCH, SOT-23_MC_MCH
- removed REF**: Battery_CR1225, Battery_CR1225
- removed REF**: MR25H40CDC_EVS, MR25H40CDC_EVS
- removed REF**: LQFP64-10x10mm, STM32F103RET6
- removed REF**: 1351-01_NXP, 1351-01_NXP
- removed REF** (x4): RES_ERJ-2GEJ103X, 0402R
- removed REF**: 61300611121, 61300611121
- removed REF** (x10): CAPC1005X55N, 0402C
- removed REF**: SW_KMR221GLFS, KMR221GLFS
- removed REF**: 0402_AVX, 0402_AVX
- removed REF**: XTAL_NX5032GA-16.000M-STD-CSU-2_NDK, NX5032GA_16_000M_STD_CSU_2
- removed REF**: 61300311121, 61300311121
- removed REF**: MIC_ICS-40720, MIC_ICS-40720
- added B1: Battery_CR1225, Battery_CR1225, F.Cu at (167.5, 78.2)
- added C1: C_0402_1005Metric, C_0402_1005Metric, F.Cu at (179.1, 114.7)
- added C10: CAPC1005X55N, 0402C, F.Cu at (153.9, 113.5)
- added C11: CAPC1005X55N, 0402C, F.Cu at (151.0, 112.9)
- added C12: CAPC1005X55N, 0402C, F.Cu at (142.4, 103.1)
- added C13: CAPC1005X55N, 0402C, F.Cu at (146.4, 91.1)
- added C14: CAPC1005X55N, 0402C, F.Cu at (155.0, 87.8)
- added C15: CAPC1005X55N, 0402C, F.Cu at (159.2, 88.5)
- added C16: YAG_CC0603_YAG, YAG_CC0603_YAG, F.Cu at (144.4, 127.8)
- added C17: YAG_CC0603_YAG, YAG_CC0603_YAG, F.Cu at (133.3, 127.4)
- added C18: CAP_CL10A105KB8NNN_SAM, CAP_CL10A105KB8NNN_SAM, F.Cu at (152.4, 90.7)
- added C19: 0402_AVX, 0402_AVX, F.Cu at (146.7, 101.6)
- added C2: C_0402_1005Metric, C_0402_1005Metric, F.Cu at (176.5, 116.9)
- added C20: CAP_0402_SAM, CAP_0402_SAM, F.Cu at (130.6, 105.2)
- added C21: C_0603_1608Metric, C_0603_1608Metric, F.Cu at (171.7, 126.2)
- added C22: CAP_0402_SAM, CAP_0402_SAM, F.Cu at (128.7, 124.6)
- added C23: C_0402_1005Metric, C_0402_1005Metric, F.Cu at (173.1, 82.1)
- added C24: C_0603_1608Metric, C_0603_1608Metric, F.Cu at (154.3, 76.2)
- added C25: C_0603_1608Metric, C_0603_1608Metric, F.Cu at (153.6, 79.3)
- added C26: C_0603_1608Metric, C_0603_1608Metric, F.Cu at (140.3, 77.1)
- added C3: C_0402_1005Metric, C_0402_1005Metric, F.Cu at (141.5, 117.5)
- added C4: C_0402_1005Metric, C_0402_1005Metric, F.Cu at (153.8, 110.8)
- added C5: SOT23-3_LTF, SOT23-3_LTF, F.Cu at (159.8, 84.4)
- added C6: CAPC1005X55N, 0402C, F.Cu at (165.0, 108.8)
- added C7: CAPC1005X55N, 0402C, F.Cu at (162.2, 111.3)
- added C8: CAPC1005X55N, 0402C, F.Cu at (159.4, 112.8)
- added C9: CAPC1005X55N, 0402C, F.Cu at (156.6, 113.4)
- added D1: SOD-123_ONS, SOD-123_ONS, F.Cu at (139.1, 121.1)
- added D2: SDO_CFP5_SOD128_NEX, SDO_CFP5_SOD128_NEX, F.Cu at (173.1, 122.2)
- added I1: SOT95P285X113-3N, SOT95P285X113-3N, F.Cu at (175.9, 78.2)
- added J1: CUI_PJ-044A, CUI_PJ-044A, F.Cu at (152.0, 122.2)
- added J2: 61300611121, 61300611121, F.Cu at (167.1, 116.7)
- added J3: 61300311121, 61300311121, F.Cu at (149.4, 85.2)
- added M1: MIC_ICS-40720, MIC_ICS-40720, F.Cu at (147.2, 76.2)
- added Q1: SOT-23_DIO, SOT-23_DIO, F.Cu at (133.6, 123.5)
- added Q2: SOT-323_DIO, SOT-323_DIO, F.Cu at (146.5, 107.8)
- added R1: R_0402_1005Metric, R_0402_1005Metric, F.Cu at (180.1, 112.1)
- added R10: RES_ERJ-2GEJ103X, 0402R, F.Cu at (167.5, 103.4)
- added R11: RES_ERJ-2GEJ103X, 0402R, F.Cu at (166.6, 106.1)
- added R12: RES_ERJ-2GEJ103X, 0402R, F.Cu at (149.2, 89.3)
- added R2: R_0402_1005Metric, R_0402_1005Metric, F.Cu at (168.4, 113.1)
- added R3: R_0603_1608Metric, R_0603_1608Metric, F.Cu at (134.5, 112.4)
- added R4: R_0402_1005Metric, R_0402_1005Metric, F.Cu at (163.5, 122.2)
- added R5: R_0402_1005Metric, R_0402_1005Metric, F.Cu at (163.2, 124.8)
- added R6: R_0402_1005Metric, R_0402_1005Metric, F.Cu at (162.3, 127.4)
- added R7: R_0402_1005Metric, R_0402_1005Metric, F.Cu at (140.7, 124.4)
- added R8: R_0402_1005Metric, R_0402_1005Metric, F.Cu at (156.6, 109.6)
- added R9: RES_ERJ-2GEJ103X, 0402R, F.Cu at (167.8, 100.7)
- added S1: SW_KMR221GLFS, KMR221GLFS, F.Cu at (145.4, 112.9)
- added U1: SOT25_DIO, SOT25_DIO, F.Cu at (174.1, 111.4)
- added U2: SOT-23_MC_MCH, SOT-23_MC_MCH, F.Cu at (133.8, 106.4)
- added U3: LQFP64-10x10mm, STM32F103RET6, F.Cu at (155.0, 100.7)
- added U4: MR25H40CDC_EVS, MR25H40CDC_EVS, F.Cu at (174.3, 92.3)
- added U5: 8L_USON_2X3_ISI, 8L_USON_2X3_ISI, F.Cu at (138.8, 127.8)
- added U6: 1351-01_NXP, 1351-01_NXP, F.Cu at (135.5, 89.2)
- added U7: MC3635_MEM, MC3635_MEM, F.Cu at (167.3, 123.5)
- added U8: BMX160_BOS, BMX160_BOS, F.Cu at (138.1, 115.3)
- added X1: XTAL_NX5032GA-16.000M-STD-CSU-2_NDK, NX5032GA_16_000M_STD_CSU_2, F.Cu at (141.3, 107.4)
Other:
- board size 40 x 40 mm -> 60 x 60 mm

Commit message: 流程适配-开始反写网表
Parts:
- moved C22 57.3 mm to (173.1, 88.4)
- moved U2 52.9 mm to (182.8, 86.4)
- moved C21 52.2 mm to (146.4, 80.5)
- moved U7 50.2 mm to (141.3, 80.5)
- moved R3 49.4 mm to (179.1, 91.3)
- moved U4 42.3 mm to (132.3, 87.3)
- moved I1 38.7 mm to (137.8, 85.1)
- moved U8 36.4 mm to (160.1, 86.3)
- moved D1 35.3 mm to (171.5, 107.0)
- moved R7 32.1 mm to (169.6, 110.3)
- moved C26 31.5 mm to (170.7, 85.4)
- moved C18 28.9 mm to (149.7, 119.4)
- moved Q1 28.7 mm to (162.0, 127.4)
- moved U5 26.8 mm to (162.8, 115.8)
- moved C16 26.8 mm to (168.4, 115.8)
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
Commit message: 流程适配-反写网表-v2
Parts:
- moved I1 54.7 mm to (178.9, 121.2)
- moved C4 53.4 mm to (169.8, 75.0)
- moved C3 47.3 mm to (167.9, 77.6)
- moved C23 42.2 mm to (176.1, 125.1)
- moved B1 40.5 mm to (170.5, 121.2)
- moved C5 40.0 mm to (173.8, 108.4)
- moved R2 39.8 mm to (136.0, 86.3)
- moved C2 37.7 mm to (135.2, 88.9)
- moved U2 37.0 mm to (147.8, 74.4)
- moved U1 35.2 mm to (141.1, 89.4)
- moved J1 35.0 mm to (178.0, 83.2)
- moved C1 34.6 mm to (135.5, 91.5)
- moved R4 34.1 mm to (179.2, 94.7)
- moved Q2 33.7 mm to (167.1, 94.1)
- moved Q1 33.4 mm to (179.1, 98.7)
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Connections:
- C1 pad 1: (no net) -> Net-(U1-IN)
- C1 pad 2: (no net) -> Net-(C1-Pad2)
- C10 pad 1: (no net) -> Net-(C9-1)
- C10 pad 2: (no net) -> Net-(C6-2)
- C11 pad 1: (no net) -> Net-(C9-1)
- C11 pad 2: (no net) -> Net-(C6-2)
- C12 pad 1: (no net) -> Net-(X1-2)
- C12 pad 2: (no net) -> Net-(C12-2)
- C13 pad 1: (no net) -> Net-(C9-1)
- C13 pad 2: (no net) -> Net-(C6-2)
- C14 pad 1: (no net) -> Net-(C9-1)
- C14 pad 2: (no net) -> Net-(C6-2)
- C15 pad 1: (no net) -> Net-(S1-P$2)
- C15 pad 2: (no net) -> Net-(S1-P$1)
- C16 pad 1: (no net) -> Net-(C16-Pad1)
- C16 pad 2: (no net) -> Net-(C17-Pad2)
- C17 pad 1: (no net) -> Net-(C16-Pad1)
- C17 pad 2: (no net) -> Net-(C17-Pad2)
- C18 pad 1: (no net) -> Net-(U6-VS)
- C18 pad 2: (no net) -> Net-(C18-Pad2)
- C19 pad 1: (no net) -> Net-(C19-Pad1)
- C19 pad 2: (no net) -> Net-(C18-Pad2)
- C2 pad 1: (no net) -> Net-(C2-Pad1)
- C2 pad 2: (no net) -> Net-(C2-Pad2)
- C20 pad 1: (no net) -> Net-(U6-VS)
- C20 pad 2: (no net) -> Net-(C18-Pad2)
- C21 pad 1: (no net) -> Net-(C21-Pad1)
- C21 pad 2: (no net) -> Net-(C21-Pad2)
- C22 pad 1: (no net) -> Net-(U8-VDDIO)
- C22 pad 2: (no net) -> Net-(C22-Pad2)
- C23 pad 1: (no net) -> Net-(B1-+)
- C23 pad 2: (no net) -> Net-(I1-GND)
- C24 pad 1: (no net) -> Net-(C24-Pad1)
- C24 pad 2: (no net) -> Net-(M1-VDD)
- C25 pad 1: (no net) -> Net-(C25-Pad1)
- C25 pad 2: (no net) -> KLT18
- C26 pad 1: (no net) -> Net-(C26-Pad1)
- C26 pad 2: (no net) -> KLT17
- C3 pad 1: (no net) -> Net-(C3-1)
- C3 pad 2: (no net) -> Net-(C3-2)
- C4 pad 1: (no net) -> Net-(D2-K)
- C4 pad 2: (no net) -> Net-(Q2-COLLECTOR)
- C5 pad 1: (no net) -> KLT14
- C5 pad 2: (no net) -> unconnected-(C5-2-Pad2)
- C5 pad 3: (no net) -> Net-(C5-3)
- C6 pad 1: (no net) -> Net-(C9-1)
- C6 pad 2: (no net) -> Net-(C6-2)
- C7 pad 1: (no net) -> Net-(C9-1)
- C7 pad 2: (no net) -> Net-(C6-2)
- C8 pad 1: (no net) -> Net-(X1-1)
- C8 pad 2: (no net) -> Net-(C8-2)
- C9 pad 1: (no net) -> Net-(C9-1)
- C9 pad 2: (no net) -> Net-(C6-2)
- D1 pad 1: (no net) -> Net-(R8-2)
- D1 pad 2: (no net) -> Net-(D1-A)
- D2 pad 1: (no net) -> Net-(D2-K)
- D2 pad 2: (no net) -> Net-(J1-Pad1)
- I1 pad 1: (no net) -> Net-(B1-+)
- I1 pad 2: (no net) -> Net-(I1-GND)
- I1 pad 3: (no net) -> Net-(I1-GND)
- J1 pad 1: (no net) -> Net-(J1-Pad1)
- J1 pad 2: (no net) -> Net-(J1-Pad2)
- J1 pad 3: (no net) -> Net-(J1-Pad2)
- J2 pad 1: (no net) -> Net-(J2-1)
- J2 pad 2: (no net) -> Net-(J2-2)
- J2 pad 3: (no net) -> Net-(J2-3)
- J2 pad 4: (no net) -> Net-(J2-4)
- J2 pad 5: (no net) -> unconnected-(J2-5-Pad5)
- J2 pad 6: (no net) -> unconnected-(J2-6-Pad6)
- J3 pad 1: (no net) -> Net-(J3-Pad1)
- J3 pad 2: (no net) -> Net-(J3-Pad2)
- J3 pad 3: (no net) -> Net-(J3-Pad3)
- M1 pad 1: (no net) -> Net-(M1-VDD)
- M1 pad 2: (no net) -> Net-(C26-Pad1)
- M1 pad 3: (no net) -> Net-(C25-Pad1)
- M1 pad 4: (no net) -> Net-(M1-GND)
- Q1 pad 1: (no net) -> Net-(R4-2)
- Q1 pad 2: (no net) -> Net-(C3-1)
- Q1 pad 3: (no net) -> Net-(D2-K)
- Q2 pad 1: (no net) -> Net-(R8-1)
- Q2 pad 2: (no net) -> Net-(D2-K)
- Q2 pad 3: (no net) -> Net-(Q2-COLLECTOR)
- R1 pad 1: (no net) -> Net-(C2-Pad1)
- R1 pad 2: (no net) -> Net-(R1-Pad2)
- R10 pad 1: (no net) -> Net-(R10-1)
- R10 pad 2: (no net) -> Net-(R10-2)
- R11 pad 1: (no net) -> Net-(R11-1)
- R11 pad 2: (no net) -> Net-(R11-2)
- R12 pad 1: (no net) -> Net-(S1-P$2)
- R12 pad 2: (no net) -> Net-(R12-2)
- R2 pad 1: (no net) -> Net-(R1-Pad2)
- R2 pad 2: (no net) -> Net-(R2-Pad2)
- R3 pad 1: (no net) -> Net-(U2-*RESET)
- R3 pad 2: (no net) -> Net-(R3-Pad2)
- R4 pad 1: (no net) -> Net-(Q2-COLLECTOR)
- R4 pad 2: (no net) -> Net-(R4-2)
- R5 pad 1: (no net) -> Net-(R5-1)
- R5 pad 2: (no net) -> Net-(Q2-COLLECTOR)
- R6 pad 1: (no net) -> Net-(Q2-COLLECTOR)
- R6 pad 2: (no net) -> Net-(D2-K)
- R7 pad 1: (no net) -> Net-(R8-2)
- R7 pad 2: (no net) -> Net-(D2-K)
- R8 pad 1: (no net) -> Net-(R8-1)
- R8 pad 2: (no net) -> Net-(R8-2)
- R9 pad 1: (no net) -> Net-(J3-Pad2)
- R9 pad 2: (no net) -> Net-(R9-2)
- S1 pad 1: (no net) -> Net-(S1-P$1)
- S1 pad 3: (no net) -> Net-(S1-P$2)
- U1 pad 1: (no net) -> Net-(U1-IN)
- U1 pad 2: (no net) -> Net-(U1-GND)
- U1 pad 3: (no net) -> Net-(U1-EN)
- U1 pad 4: (no net) -> Net-(R1-Pad2)
- U1 pad 5: (no net) -> Net-(C2-Pad1)
- U2 pad 1: (no net) -> Net-(U2-VDD)
- U2 pad 2: (no net) -> Net-(U2-GND)
- U2 pad 3: (no net) -> Net-(U2-*RESET)
- U3 pad 1: (no net) -> Net-(U3-VBAT)
- U3 pad 10: (no net) -> KLT18
- U3 pad 11: (no net) -> KLT17
- U3 pad 12: (no net) -> Net-(U3-VSS)
- U3 pad 13: (no net) -> Net-(U3-VDDA)
- U3 pad 14: (no net) -> KLT16
- U3 pad 15: (no net) -> KLT15
- U3 pad 16: (no net) -> KLT14
- U3 pad 17: (no net) -> KLT13
- U3 pad 18: (no net) -> Net-(U3-VSS)
- U3 pad 19: (no net) -> Net-(U3-VDDA)
- U3 pad 2: (no net) -> KLT12
- U3 pad 20: (no net) -> KLT11
- U3 pad 21: (no net) -> KLT10
- U3 pad 22: (no net) -> KLT9
- U3 pad 23: (no net) -> KLT8
- U3 pad 24: (no net) -> KLT7
- U3 pad 25: (no net) -> KLT6
- U3 pad 26: (no net) -> KLT5
- U3 pad 27: (no net) -> KLT4
- U3 pad 28: (no net) -> KLT3
- U3 pad 29: (no net) -> I2C_SCL
- U3 pad 3: (no net) -> KLT2
- U3 pad 30: (no net) -> I2C_SDA
- U3 pad 31: (no net) -> Net-(U3-VSS)
- U3 pad 32: (no net) -> Net-(U3-VDDA)
- U3 pad 33: (no net) -> KLT1
- U3 pad 34: (no net) -> KLT0
- U3 pad 35: (no net) -> Net-(U3-PB14)
- U3 pad 36: (no net) -> Net-(U3-PB15)
- U3 pad 37: (no net) -> Net-(U3-PC6)
- U3 pad 38: (no net) -> Net-(U3-PC7)
- U3 pad 39: (no net) -> Net-(U3-PC8)
- U3 pad 4: (no net) -> Net-(U3-PC15-_OSC32_OUT)
- U3 pad 40: (no net) -> Net-(U3-PC9)
- U3 pad 41: (no net) -> Net-(U3-PA8)
- U3 pad 42: (no net) -> Net-(U3-PA9)
- U3 pad 43: (no net) -> Net-(U3-PA10)
- U3 pad 44: (no net) -> Net-(U3-PA11)
- U3 pad 45: (no net) -> Net-(U3-PA12)
- U3 pad 46: (no net) -> Net-(J2-3)
- U3 pad 47: (no net) -> Net-(U3-VSS)
- U3 pad 48: (no net) -> Net-(U3-VDDA)
- U3 pad 49: (no net) -> Net-(J2-2)
- U3 pad 5: (no net) -> Net-(X1-2)
- U3 pad 50: (no net) -> SPI0_CSN
- U3 pad 51: (no net) -> Net-(U3-PC10)
- U3 pad 52: (no net) -> Net-(U3-PC11)
- U3 pad 53: (no net) -> Net-(U3-PC12)
- U3 pad 54: (no net) -> Net-(U3-PD2)
- U3 pad 55: (no net) -> SPI_SCK
- U3 pad 56: (no net) -> SPI_MISO
- U3 pad 57: (no net) -> SPI_MOSI
- U3 pad 58: (no net) -> Net-(R11-1)
- U3 pad 59: (no net) -> Net-(R10-1)
- U3 pad 6: (no net) -> Net-(X1-1)
- U3 pad 60: (no net) -> Net-(R9-2)
- U3 pad 61: (no net) -> Net-(U3-PB8)
- U3 pad 62: (no net) -> Net-(U3-PB9)
- U3 pad 63: (no net) -> Net-(U3-VSS)
- U3 pad 64: (no net) -> Net-(U3-VDDA)
- U3 pad 7: (no net) -> Net-(S1-P$2)
- U3 pad 8: (no net) -> Net-(U3-PC0)
- U3 pad 9: (no net) -> Net-(U3-PC1)
- U4 pad 1: (no net) -> KLT0
- U4 pad 2: (no net) -> KLT1
- U4 pad 3: (no net) -> KLT2
- U4 pad 4: (no net) -> Net-(U4-VSS)
- U4 pad 5: (no net) -> KLT3
- U4 pad 6: (no net) -> KLT4
- U4 pad 7: (no net) -> KLT5
- U4 pad 8: (no net) -> Net-(U4-VDD)
- U5 pad 1: (no net) -> KLT6
- U5 pad 2: (no net) -> KLT7
- U5 pad 3: (no net) -> KLT8
- U5 pad 4: (no net) -> Net-(U5-GND)
- U5 pad 5: (no net) -> KLT9
- U5 pad 6: (no net) -> KLT10
- U5 pad 7: (no net) -> KLT11
- U5 pad 8: (no net) -> Net-(U5-VCC)
- U5 pad 9: (no net) -> Net-(U5-GND)
- U6 pad 2: (no net) -> Net-(U6-VS)
- U6 pad 3: (no net) -> Net-(C18-Pad2)
- U6 pad 4: (no net) -> Net-(C19-Pad1)
- U7 pad 1: (no net) -> Net-(U7-DOUT_A1)
- U7 pad 10: (no net) -> I2C_SCL
- U7 pad 2: (no net) -> I2C_SDA
- U7 pad 4: (no net) -> Net-(U7-VPP)
- U7 pad 5: (no net) -> KLT16
- U7 pad 6: (no net) -> Net-(U7-VDD)
- U7 pad 7: (no net) -> Net-(U7-VDD)
- U7 pad 8: (no net) -> Net-(U7-VPP)
- U7 pad 9: (no net) -> Net-(U7-CSN)
- U8 pad 1: (no net) -> SPI_MISO
- U8 pad 10: (no net) -> unconnected-(U8-DNC-Pad10)
- U8 pad 11: (no net) -> unconnected-(U8-DNC-Pad11)
- U8 pad 12: (no net) -> SPI0_CSN
- U8 pad 13: (no net) -> SPI_SCK
- U8 pad 14: (no net) -> SPI_MOSI
- U8 pad 2: (no net) -> Net-(U8-GND)
- U8 pad 3: (no net) -> Net-(U8-GND)
- U8 pad 4: (no net) -> KLT12
- U8 pad 5: (no net) -> Net-(U8-VDDIO)
- U8 pad 6: (no net) -> Net-(C22-Pad2)
- U8 pad 7: (no net) -> Net-(C22-Pad2)
- U8 pad 8: (no net) -> Net-(U8-VDD)
- U8 pad 9: (no net) -> KLT13
- X1 pad 1: (no net) -> Net-(X1-1)
- X1 pad 2: (no net) -> Net-(X1-2)
