File: app/services/layout_service/data/temp/project/Project.kicad_sch (KiCad schematic)
At the start: 22 parts, among them J1 AU-Y1007, U1 TCM809RVNB713, U2 ATTINY1626-MUR, X1 12 MHz

Commit message: 动态适配本地板子-2.2
Parts:
- removed C1, C6: 10uF, ATTINY1626_MUR:C_0402_1005Metric, symbol d2e61be6e8d5431b80327900143beec2
- removed C2, C8: 0.1uF, ATTINY1626_MUR:C_0402_1005Metric, symbol d679d6ad08804ffe98034658b412e359
- removed C5: 10pF, ATTINY1626_MUR:C_0402_1005Metric, symbol 85d13148a64c4414bd71c9d86d11548f
- removed L1: LTST-C191KSKT, LTST-C191KSKT:LED_LTST-C191KRKT_LTO, symbol 2024-07-24_02-14-48:LTST-C191KSKT
- removed R3: 300, LTST-C191KSKT:R_0603_1608Metric, symbol dddccab79a8e42babc2b4fe9f24879e9
- removed R5: 330, ATTINY1626_MUR:R_0402_1005Metric, symbol c67428543f594619a0dd718329961ce6
- removed R6: 10k, ATTINY1626_MUR:R_0402_1005Metric, symbol 5b03a4e39cdd44388ac81e5147c6d544
- removed U1: TCM809RVNB713, TCM809:SOT-23_MC_MCH, symbol 2024-07-15_06-27-23:TCM809RVNB713
- removed U2: ATTINY1626-MUR, ATTINY1626_MUR:QFN40P300X300X90-21N, symbol ATTINY1626_MUR:ATTINY1626-MUR
- added C1: 1.5uF, MAX6703ARKA+:C_0603_1608Metric, symbol Device:C
- added C10, C12: 10uF, ATSAMD21G18A-MUT:0603C, symbol d2e61be6e8d5431b80327900143beec2
- added C11, C6: 12 pF, ATSAMD21G18A-MUT:0402C, symbol 8eea43a4825740aab88bcdde5055dec8
- added C2: 10 pF, ATSAMD21G18A-MUT:0402C, symbol 85d13148a64c4414bd71c9d86d11548f
- added C5, C9: 0.1uF, ATSAMD21G18A-MUT:0402C, symbol d679d6ad08804ffe98034658b412e359
- added C8: 1uF, ATSAMD21G18A-MUT:0402C, symbol 055cae77582c4e138823cacd5dfe841c
- added J2: M50-3500542, ATSAMD21G18A-MUT:M50_3500542, symbol f5efde0bca2a441da320adfe9e5c3236
- added L1: 150080GS75000, LED_GS75000_WRE, symbol 2024-07-24_03-11-48:150080GS75000
- added R10: 10k, ATSAMD21G18A-MUT:0402R, symbol 5b03a4e39cdd44388ac81e5147c6d544
- added R3: 300, 150080GS75000:R_0603_1608Metric, symbol c34b79a2ac99493299f236e6c9775f0f
- added R5, R6: 4.7k, ATSAMD21G18A-MUT:0402R, symbol 59d8dd5d3684403883a6edf3276d16f2
- added R8: 1k, ATSAMD21G18A-MUT:0402R, symbol eef5dda9063344d2ac8d765518fca3c7
- added R9: 330, ATSAMD21G18A-MUT:0402R, symbol c67428543f594619a0dd718329961ce6
- added U1: MAX6421XS29+T, MAX6703ARKA+:21-0098_X4&plus_1_MXM, symbol 2024-07-25_00-58-29:MAX6421XS29+T
- added U2: ATSAMD21G18A-MUT, ATSAMD21G18A-MUT:QFN48_7X7MC_MCH, symbol a694860fc00444b8bf70d6151e701455
- added X2: 32.768 kHz, ATSAMD21G18A-MUT:ABS05_32_768KHZ_T, symbol b288647140ea4bdb87abf4ea1a6ef720
- C3, C4: footprint ATTINY1626_MUR:C_0402_1005Metric -> ATSAMD21G18A-MUT:0402C
- C7: value 10pF -> 10 pF; footprint ATTINY1626_MUR:C_0402_1005Metric -> ATSAMD21G18A-MUT:0402C
- R1: value 100K -> 100k; footprint TCM809:R_0603_1608Metric -> MAX6703ARKA+:RC0805N_YAG
- R4, R7: footprint ATTINY1626_MUR:R_0402_1005Metric -> ATSAMD21G18A-MUT:0402R
- S2: footprint ATTINY1626_MUR:B3U-1000P -> ATSAMD21G18A-MUT:B3U-1000P
- X1: footprint ATTINY1626_MUR:ABM8G_12_000MHZ_B4Y_T -> ATSAMD21G18A-MUT:ABM8G_12_000MHZ_B4Y_T
Connections:
- net 3V3: now also C4.1, C10.1, C12.1, C5.1, J2.1, R10.2, R5.2, R6.2, R8.2, U1.1 (VCC), U2.17 (VDDIO), U2.36 (VDDIO), U2.44 (VDDIN), U2.6 (VDDANA)
- net GND: now also C1.2, C10.2, C11.2, C12.2, C2.2, C5.2, C6.2, C8.2, C9.2, J2.3, J2.5, L1.1, U1.2 (GND), U2.18 (GND), U2.35 (GND), U2.42 (GND), U2.49 (EP_GND), U2.5 (GNDANA)
- net at R4.1: now also U2.25 (PA16)
- net at X1.1 (IN/OUT): now also C7.1
- net at X1.3 (OUT/IN): now also C2.1; no longer C7.1
- net at R7.1: now also U2.26 (PA17)
- net at S2.2: now also R9.2
- net KLT_1_PA7 renamed KLT_1_XIN32
- net KLT_1_XIN32: now also C6.1, U1.4 (*RESET), U2.1 (PA00), X2.1
- net KLT_2_PA2 renamed KLT_2_PA05
- net KLT_2_PA05: now also U2.10 (PA05)
- net KLT_3_PB4 renamed KLT_4_PA07
- net KLT_4_PA07: now also U2.12 (PA07)
- net KLT_4_PC1 renamed KLT_5_PA08
- net KLT_5_PA08: now also U2.13 (PA08)
- new net: L1.2, R3.1
- new net: R6.1, U2.31 (PA22)
- new net: R5.1, U2.32 (PA23)
- new net: C8.1, U2.43 (VDDCORE)
- new net: C1.1, U1.3 (SRT)
- new net: J2.4, R8.1
- new net: C9.1, R10.1, R9.1
- new net: C11.1, X2.2
- new net KLT_3_PA06: R3.2, U2.11 (PA06)
- no-connect marks 13 -> 45
Other:
- note added: "电源监控器 （Power Monitor）"
- note removed: "电源监控器 (Power Monitor)"
- title: KLT_设计_1891296611015680002 -> KLT_设计_1889969586090893314
- moved on the sheet: J1, R2, S1
