File: app/services/layout_service/data/temp/template/project.kicad_pcb (KiCad board)
At the start: 2 copper layers, 40 x 40 mm, 58 parts

Commit message: 流程适配-开始考虑焊盘和旋转
Parts:
- removed IC**: SOT95P285X113-3N, SOT95P285X113-3N
- removed REF** (x4): C_0603_1608Metric, C_0603_1608Metric
- removed REF**: 8L_USON_2X3_ISI, 8L_USON_2X3_ISI
- removed REF** (x2): YAG_CC0603_YAG, YAG_CC0603_YAG
- removed REF** (x2): CAP_0402_SAM, CAP_0402_SAM
- removed REF**: BMX160_BOS, BMX160_BOS
- removed REF**: SOT23-3_LTF, SOT23-3_LTF
- removed REF** (x7): R_0402_1005Metric, R_0402_1005Metric
- removed REF** (x5): C_0402_1005Metric, C_0402_1005Metric
- removed REF**: MC3635_MEM, MC3635_MEM
- removed REF**: SOT25_DIO, SOT25_DIO
- removed REF**: SOD-123_ONS, SOD-123_ONS
- removed REF**: CUI_PJ-044A, CUI_PJ-044A
- removed REF**: SDO_CFP5_SOD128_NEX, SDO_CFP5_SOD128_NEX
- removed REF**: CAP_CL10A105KB8NNN_SAM, CAP_CL10A105KB8NNN_SAM
- removed REF**: SOT-23_DIO, SOT-23_DIO
- removed REF**: SOT-323_DIO, SOT-323_DIO
- removed REF**: R_0603_1608Metric, R_0603_1608Metric
- removed REF**: SOT-23_MC_MCH, SOT-23_MC_MCH
- removed REF**: Battery_CR1225, Battery_CR1225
- removed REF**: MR25H40CDC_EVS, MR25H40CDC_EVS
- removed REF**: LQFP64-10x10mm, STM32F103RET6
- removed REF**: 1351-01_NXP, 1351-01_NXP
- removed REF** (x4): RES_ERJ-2GEJ103X, 0402R
- removed REF**: 61300611121, 61300611121
- removed REF** (x10): CAPC1005X55N, 0402C
- removed REF**: SW_KMR221GLFS, KMR221GLFS
- removed REF**: 0402_AVX, 0402_AVX
- removed REF**: XTAL_NX5032GA-16.000M-STD-CSU-2_NDK, NX5032GA_16_000M_STD_CSU_2
- removed REF**: 61300311121, 61300311121
- removed REF**: MIC_ICS-40720, MIC_ICS-40720
- added B1: Battery_CR1225, Battery_CR1225, F.Cu at (0.00, 0.00)
- added C1, C2, C23, C3, C4: C_0402_1005Metric, C_0402_1005Metric, F.Cu at (0.00, 0.00)
- added C10, C11, C12, C13, C14, C15, C6, C7, C8, C9: CAPC1005X55N, 0402C, F.Cu at (0.00, 0.00)
- added C16, C17: YAG_CC0603_YAG, YAG_CC0603_YAG, F.Cu at (0.00, 0.00)
- added C18: CAP_CL10A105KB8NNN_SAM, CAP_CL10A105KB8NNN_SAM, F.Cu at (0.00, 0.00)
- added C19: 0402_AVX, 0402_AVX, F.Cu at (0.00, 0.00)
- added C20, C22: CAP_0402_SAM, CAP_0402_SAM, F.Cu at (0.00, 0.00)
- added C21, C24, C25, C26: C_0603_1608Metric, C_0603_1608Metric, F.Cu at (0.00, 0.00)
- added C5: SOT23-3_LTF, SOT23-3_LTF, F.Cu at (0.00, 0.00)
- added D1: SOD-123_ONS, SOD-123_ONS, F.Cu at (0.00, 0.00)
- added D2: SDO_CFP5_SOD128_NEX, SDO_CFP5_SOD128_NEX, F.Cu at (0.00, 0.00)
- added I1: SOT95P285X113-3N, SOT95P285X113-3N, F.Cu at (0.00, 0.00)
- added J1: CUI_PJ-044A, CUI_PJ-044A, F.Cu at (0.00, 0.00)
- added J2: 61300611121, 61300611121, F.Cu at (0.00, 0.00)
- added J3: 61300311121, 61300311121, F.Cu at (0.00, 0.00)
- added M1: MIC_ICS-40720, MIC_ICS-40720, F.Cu at (0.00, 0.00)
- added Q1: SOT-23_DIO, SOT-23_DIO, F.Cu at (0.00, 0.00)
- added Q2: SOT-323_DIO, SOT-323_DIO, F.Cu at (0.00, 0.00)
- added R1, R2, R4, R5, R6, R7, R8: R_0402_1005Metric, R_0402_1005Metric, F.Cu at (0.00, 0.00)
- added R10, R11, R12, R9: RES_ERJ-2GEJ103X, 0402R, F.Cu at (0.00, 0.00)
- added R3: R_0603_1608Metric, R_0603_1608Metric, F.Cu at (0.00, 0.00)
- added S1: SW_KMR221GLFS, KMR221GLFS, F.Cu at (0.00, 0.00)
- added U1: SOT25_DIO, SOT25_DIO, F.Cu at (0.00, 0.00)
- added U2: SOT-23_MC_MCH, SOT-23_MC_MCH, F.Cu at (0.00, 0.00)
- added U3: LQFP64-10x10mm, STM32F103RET6, F.Cu at (0.00, 0.00)
- added U4: MR25H40CDC_EVS, MR25H40CDC_EVS, F.Cu at (0.00, 0.00)
- added U5: 8L_USON_2X3_ISI, 8L_USON_2X3_ISI, F.Cu at (0.00, 0.00)
- added U6: 1351-01_NXP, 1351-01_NXP, F.Cu at (0.00, 0.00)
- added U7: MC3635_MEM, MC3635_MEM, F.Cu at (0.00, 0.00)
- added U8: BMX160_BOS, BMX160_BOS, F.Cu at (0.00, 0.00)
- added X1: XTAL_NX5032GA-16.000M-STD-CSU-2_NDK, NX5032GA_16_000M_STD_CSU_2, F.Cu at (0.00, 0.00)
Other:
- board outline removed

Commit message: 流程适配完成-v1.0
Parts:
- removed B1: Battery_CR1225, Battery_CR1225
- removed C10, C11, C12, C13, C14, C15, C9: CAPC1005X55N, 0402C
- removed C16, C17: YAG_CC0603_YAG, YAG_CC0603_YAG
- removed C18: CAP_CL10A105KB8NNN_SAM, CAP_CL10A105KB8NNN_SAM
- removed C19: 0402_AVX, 0402_AVX
- removed C20, C22: CAP_0402_SAM, CAP_0402_SAM
- removed C21, C24, C25, C26: C_0603_1608Metric, C_0603_1608Metric
- removed C23: C_0402_1005Metric, C_0402_1005Metric
- removed D1: SOD-123_ONS, SOD-123_ONS
- removed D2: SDO_CFP5_SOD128_NEX, SDO_CFP5_SOD128_NEX
- removed I1: SOT95P285X113-3N, SOT95P285X113-3N
- removed J2: 61300611121, 61300611121
- removed J3: 61300311121, 61300311121
- removed M1: MIC_ICS-40720, MIC_ICS-40720
- removed Q1: SOT-23_DIO, SOT-23_DIO
- removed Q2: SOT-323_DIO, SOT-323_DIO
- removed R10, R11, R12, R9: RES_ERJ-2GEJ103X, 0402R
- removed R8: R_0402_1005Metric, R_0402_1005Metric
- removed U3: LQFP64-10x10mm, STM32F103RET6
- removed U4: MR25H40CDC_EVS, MR25H40CDC_EVS
- removed U5: 8L_USON_2X3_ISI, 8L_USON_2X3_ISI
- removed U6: 1351-01_NXP, 1351-01_NXP
- removed U7: MC3635_MEM, MC3635_MEM
- removed U8: BMX160_BOS, BMX160_BOS
- added L1: LED_LTST-C191KRKT_LTO, LED_LTST-C191KRKT_LTO, F.Cu at (0.00, 0.00)
- added S2: B3U-1000P, B3U-1000P, F.Cu at (0.00, 0.00)
- C5: value SOT23-3_LTF -> C_0402_1005Metric; footprint SOT23-3_LTF -> C_0402_1005Metric
- C6, C7, C8: value CAPC1005X55N -> C_0402_1005Metric; footprint 0402C -> C_0402_1005Metric
- J1: value CUI_PJ-044A -> ASSMANN_AU-Y1007; footprint CUI_PJ-044A -> ASSMANN_AU-Y1007
- R1: value R_0402_1005Metric -> R_0603_1608Metric; footprint R_0402_1005Metric -> R_0603_1608Metric
- R2: value R_0402_1005Metric -> RC0402N_PAN; footprint R_0402_1005Metric -> RC0402N_PAN
- S1: value SW_KMR221GLFS -> SW_25816_WRE; footprint KMR221GLFS -> SW_25816_WRE
- U1: value SOT25_DIO -> SOT-23_MC_MCH; footprint SOT25_DIO -> SOT-23_MC_MCH
- U2: value SOT-23_MC_MCH -> QFN40P300X300X90-21N; footprint SOT-23_MC_MCH -> QFN40P300X300X90-21N
- X1: value XTAL_NX5032GA-16.000M-STD-CSU-2_NDK -> CRYSTAL_ABM8G_ABR; footprint NX5032GA_16_000M_STD_CSU_2 -> ABM8G_12_000MHZ_B4Y_T

Commit message: 动态适配本地板子-2.2
Parts:
- added C10, C12: CAPC1608X100N, 0603C, F.Cu at (0.00, 0.00)
- added C11, C9: CAPC1005X55N, 0402C, F.Cu at (0.00, 0.00)
- added J2: CONN10_500542_HRW, M50_3500542, F.Cu at (0.00, 0.00)
- added R10, R8, R9: RES_ERJ-2GEJ103X, 0402R, F.Cu at (0.00, 0.00)
- added X2: XTAL_ABS05-32.768KHZ-T, ABS05_32_768KHZ_T, F.Cu at (0.00, 0.00)
- C1: value C_0402_1005Metric -> C_0603_1608Metric; footprint C_0402_1005Metric -> C_0603_1608Metric
- C2, C3, C4, C5, C6, C7, C8: value C_0402_1005Metric -> CAPC1005X55N; footprint C_0402_1005Metric -> 0402C
- L1: value LED_LTST-C191KRKT_LTO -> LED_GS75000_WRE; footprint LED_LTST-C191KRKT_LTO -> LED_GS75000_WRE
- R1: value R_0603_1608Metric -> RC0805N_YAG; footprint R_0603_1608Metric -> RC0805N_YAG
- R4, R5, R6, R7: value R_0402_1005Metric -> RES_ERJ-2GEJ103X; footprint R_0402_1005Metric -> 0402R
- U1: value SOT-23_MC_MCH -> 21-0098_X4+1_MXM; footprint SOT-23_MC_MCH -> 21-0098_X4&plus_1_MXM
- U2: value QFN40P300X300X90-21N -> QFN48_7X7MC_MCH; footprint QFN40P300X300X90-21N -> QFN48_7X7MC_MCH
